File: CTS-SAT-1 Hardware/External Connectors.kicad_sch (KiCad schematic)
At the start: 99 parts, among them J10 J-0530471010, J11 J-0532610671, J12 J-0532610871, J14 J-0532610471, J15 J-0532610471, J2 J-TSW-106-05-T-S, J3 J-0532610871, J4 J-0532610471, J5 J-ESQ-126-14-G-D, J6 J-ESQ-126-14-G-D, J7 J-0532610671, J8 J-0532610471, J9 J-0532610471, U10 MAX3086EESD+T, U9 U-MAX3378EEUD+T

Commit message: Remove extraneous objects
Removed: FRAM, PC104 pull-downs, Altium data
Parts:
- removed R100, R101, R102, R103, R104, R105, R106, R108, R110, R111, R112, R113, R114, R115, R116, R118, R119, R120, R121, R122, R123, R124, R125, R127, R132, R133, R139, R140, R141, R94, R95, R96, R97, R98, R99: 100K, 0603, symbol OBC Development Board:root_0_RT-100K0-F-1/16W-0603_OBC Development Board.SchLib
Connections:
- net at J6.18: no longer J6.20
- net at J6.26: no longer J6.30
- net at J6.25: no longer J6.29
- net at J6.17: no longer J6.19
- now unconnected: J5.1, J5.10, J5.11, J5.12, J5.13, J5.14, J5.2, J5.3, J5.33, J5.34, J5.35, J5.36, J5.37, J5.38, J5.4, J5.5, J5.6, J5.7, J5.8, J5.9, J6.33, J6.34, J6.35, J6.36, J6.37, J6.38
- no-connect marks 17 -> 16
Other:
- note removed: "${##}"
- note removed: "${#}"
- note removed: "${ADDRESS1}"
- note removed: "${ADDRESS2}"
- note removed: "${ADDRESS3}"
- note removed: "${ADDRESS4}"
- note removed: "${CAGE_CODE}"
- note removed: "${CHECKEDBY}"
- note removed: "${CHK_APP_DATE}"
- note removed: "${DOC_NO_BOM}"
- note removed: "${DOC_NO_FAB_DWG}"
- note removed: "${DOC_NO_SCH_DWG}"
- note removed: "${DRAWNBY}"
- note removed: "${DSN_APP_DATE}"
- note removed: "${ENGINEER}"
- note removed: "${ENG_APP_DATE}"
- note removed: "${FILENAME}"
- note removed: "${ITEM}"
- note removed: "${PCB_DWG_NO}"
- note removed: "${PROJECT}"
- note removed: "${SCH_SCALE}"
- note removed: "${TITLE}"
- note removed: "${VERSIONCONTROL_PROJFOLDERREVNUMBER}"
- note removed: "${VERSIONCONTROL_REVNUMBER}"
- note removed: "1"
- note removed: "4"
- note removed: "A3"
- note removed: "APPROVALS"
- note removed: "ASSY DWG:"
- note removed: "BOM:"
- note removed: "CAGE CODE"
- note removed: "CHK:"
- note removed: "DESIGN ITEM:"
- note removed: "DOCUMENT REVISION:"
- note removed: "DSN:"
- note removed: "DWG NO."
- note removed: "External Connectors"
- note removed: "FAB DWG:"
- note removed: "FILE NAME"
- note removed: "James Chen"
- note removed: "OF"
- note removed: "PCB DWG:"
- note removed: "PROJECT"
- note removed: "PROJECT REVISION:"
- note removed: "REFERENCE DOCUMENTS"
- note removed: "REV"
- note removed: "Rev1.4"
- note removed: "SCALE:"
- note removed: "SHEET"
- note removed: "SIZE"
- note removed: "TITLE"
- moved on the sheet: C29, C30, C31, C32, J10, J4, R11, R130, R131, R64, R72, R73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
