File: Hardware/stm32_flash.kicad_sch (KiCad schematic)
At the start: 20 parts, among them IC2 MT29F1G01ABAFDSF-AAT_F_TR, IC3 MT29F1G01ABAFDSF-AAT_F_TR, IC4 MT29F1G01ABAFDSF-AAT_F_TR, IC5 MT29F1G01ABAFDSF-AAT_F_TR

Commit message: Finish schematic v1
Parts:
- renumbered R73 to R72, R74 to R73, R75 to R74, R76 to R75, R77 to R76, R78 to R77, R79 to R78, R80 to R79, R81 to R80, R82 to R81, R83 to R82, R84 to R83
Changed lines of the file:
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@@
 		(dnp no)
 		(fields_autoplaced yes)
-		(property "Reference" "#PWR099"
+		(property "Reference" "#PWR0100"
 			(at 149.86 227.33 0)
 			(effects
@@
 			(project "CTS-SAT-2-OBC-PCB"
 				(path "/58243925-df8d-4fc1-899e-fce866d1d25a/1b38ac1a-71db-4ef7-b830-b2f3080e4569"
-					(reference "#PWR099")
+					(reference "#PWR0100")
 					(unit 1)
 				)
@@
 		(on_board yes)
 		(dnp no)
-		(property "Reference" "#PWR084"
+		(property "Reference" "#PWR085"
 			(at 87.63 107.95 0)
 			(effects
@@
 			(project "CTS-SAT-2-OBC-PCB"
 				(path "/58243925-df8d-4fc1-899e-fce866d1d25a/1b38ac1a-71db-4ef7-b830-b2f3080e4569"
-					(reference "#PWR084")
+					(reference "#PWR085")
 					(unit 1)
 				)
@@
 		(on_board yes)
 		(dnp no)
-		(property "Reference" "R79"
+		(property "Reference" "R78"
 			(at 97.282 189.992 90)
 			(effects
@@
 			(project "CTS-SAT-2-OBC-PCB"
 				(path "/58243925-df8d-4fc1-899e-fce866d1d25a/1b38ac1a-71db-4ef7-b830-b2f3080e4569"
-					(reference "R79")
+					(reference "R78")
 					(unit 1)
 				)
@@
 		(dnp no)
 		(fields_autoplaced yes)
-		(property "Reference" "#PWR089"
+		(property "Reference" "#PWR090"
 			(at 93.98 130.81 0)
 			(effects
@@
 			(project "CTS-SAT-2-OBC-PCB"
 				(path "/58243925-df8d-4fc1-899e-fce866d1d25a/1b38ac1a-71db-4ef7-b830-b2f3080e4569"
-					(reference "#PWR089")
+					(reference "#PWR090")
 					(unit 1)
 				)
@@
 		(dnp no)
 		(fields_autoplaced yes)
-		(property "Reference" "R75"
+		(property "Reference" "R74"
 			(at 101.6 176.5299 0)
 			(effects
@@
 			(project "CTS-SAT-2-OBC-PCB"
 				(path "/58243925-df8d-4fc1-899e-fce866d1d25a/1b38ac1a-71db-4ef7-b830-b2f3080e4569"
-					(reference "R75")
+					(reference "R74")
 					(unit 1)
 				)
@@
 		(dnp no)
 		(fields_autoplaced yes)
-		(property "Reference" "R76"
+		(property "Reference" "R75"
 			(at 101.6 215.8999 0)
 			(effects
@@
 			(project "CTS-SAT-2-OBC-PCB"
 				(path "/58243925-df8d-4fc1-899e-fce866d1d25a/1b38ac1a-71db-4ef7-b830-b2f3080e4569"
-					(reference "R76")
+					(reference "R75")
 					(unit 1)
 				)
@@
 		(on_board yes)
 		(dnp no)
-		(property "Reference" "R80"
+		(property "Reference" "R79"
 			(at 97.282 229.362 90)
 			(effects
@@
 			(project "CTS-SAT-2-OBC-PCB"
 				(path "/58243925-df8d-4fc1-899e-fce866d1d25a/1b38ac1a-71db-4ef7-b830-b2f3080e4569"
-					(reference "R80")
+					(reference "R79")
 					(unit 1)
 				)
@@
 		(dnp no)
 		(fields_autoplaced yes)
-		(property "Reference" "#PWR092"
+		(property "Reference" "#PWR093"
 			(at 160.02 106.68 0)
 			(effects
@@
 			(project "CTS-SAT-2-OBC-PCB"
 				(path "/58243925-df8d-4fc1-899e-fce866d1d25a/1b38ac1a-71db-4ef7-b830-b2f3080e4569"
-					(reference "#PWR092")
+					(reference "#PWR093")
 					(unit 1)
 				)
@@
 		(dnp no)
 		(fields_autoplaced yes)
-		(property "Reference" "R73"
+		(property "Reference" "R72"
 			(at 101.6 97.7899 0)
 			(effects
@@
 			(project "CTS-SAT-2-OBC-PCB"
 				(path "/58243925-df8d-4fc1-899e-fce866d1d25a/1b38ac1a-71db-4ef7-b830-b2f3080e4569"
-					(reference "R73")
+					(reference "R72")
 					(unit 1)
 				)
@@
 		(on_board yes)
 		(dnp no)
-		(property "Reference" "R82"
+		(property "Reference" "R81"
 			(at 145.288 149.352 90)
 			(effects
@@
 			(project "CTS-SAT-2-OBC-PCB"
 				(path "/58243925-df8d-4fc1-899e-fce866d1d25a/1b38ac1a-71db-4ef7-b830-b2f3080e4569"
-					(reference "R82")
+					(reference "R81")
 					(unit 1)
 				)
@@
 		(dnp no)
 		(fields_autoplaced yes)
-		(property "Reference" "#PWR094"
+		(property "Reference" "#PWR095"
 			(at 160.02 144.78 0)
 			(effects
@@
 			(project "CTS-SAT-2-OBC-PCB"
 				(path "/58243925-df8d-4fc1-899e-fce866d1d25a/1b38ac1a-71db-4ef7-b830-b2f3080e4569"
-					(reference "#PWR094")
+					(reference "#PWR095")
 					(unit 1)
 				)
@@
 		(dnp no)
 		(fields_autoplaced yes)
-		(property "Reference" "#PWR088"
+		(property "Reference" "#PWR089"
 			(at 93.98 92.71 0)
 			(effects
@@
 			(project "CTS-SAT-2-OBC-PCB"
 				(path "/58243925-df8d-4fc1-899e-fce866d1d25a/1b38ac1a-71db-4ef7-b830-b2f3080e4569"
-					(reference "#PWR088")
+					(reference "#PWR089")
 					(unit 1)
 				)
@@
 		(on_board yes)
 		(dnp no)
-		(property "Reference" "R84"
+		(property "Reference" "R83"
 			(at 145.288 229.362 90)
 			(effects
@@
 			(project "CTS-SAT-2-OBC-PCB"
 				(path "/58243925-df8d-4fc1-899e-fce866d1d25a/1b38ac1a-71db-4ef7-b830-b2f3080e4569"
-					(reference "R84")
+					(reference "R83")
 					(unit 1)
 				)
@@
 		(on_board yes)
 		(dnp no)
-		(property "Reference" "R83"
+		(property "Reference" "R82"
 			(at 145.288 189.992 90)
 			(effects
@@
 			(project "CTS-SAT-2-OBC-PCB"
 				(path "/58243925-df8d-4fc1-899e-fce866d1d25a/1b38ac1a-71db-4ef7-b830-b2f3080e4569"
-					(reference "R83")
+					(reference "R82")
 					(unit 1)
 				)
@@
 		(dnp no)
 		(fields_autoplaced yes)
-		(property "Reference" "#PWR098"
+		(property "Reference" "#PWR099"
 			(at 160.02 224.79 0)
 			(effects
@@
 			(project "CTS-SAT-2-OBC-PCB"
 				(path "/58243925-df8d-4fc1-899e-fce866d1d25a/1b38ac1a-71db-4ef7-b830-b2f3080e4569"
-					(reference "#PWR098")
+					(reference "#PWR099")
 					(unit 1)
 				)
@@
 		(on_board yes)
 		(dnp no)
-		(property "Reference" "#PWR085"
+		(property "Reference" "#PWR086"
 			(at 87.63 146.05 0)
 			(effects
@@
 			(project "CTS-SAT-2-OBC-PCB"
 				(path "/58243925-df8d-4fc1-899e-fce866d1d25a/1b38ac1a-71db-4ef7-b830-b2f3080e4569"
-					(reference "#PWR085")
+					(reference "#PWR086")
 					(unit 1)
 				)
@@
 		(dnp no)
 		(fields_autoplaced yes)
-		(property "Reference" "#PWR095"
+		(property "Reference" "#PWR096"
 			(at 149.86 147.32 0)
 			(effects
@@
 			(project "CTS-SAT-2-OBC-PCB"
 				(path "/58243925-df8d-4fc1-899e-fce866d1d25a/1b38ac1a-71db-4ef7-b830-b2f3080e4569"
-					(reference "#PWR095")
+					(reference "#PWR096")
 					(unit 1)
 				)
@@
 		(dnp no)
 		(fields_autoplaced yes)
-		(property "Reference" "R74"
+		(property "Reference" "R73"
 			(at 101.6 135.8899 0)
 			(effects
@@
 			(project "CTS-SAT-2-OBC-PCB"
 				(path "/58243925-df8d-4fc1-899e-fce866d1d25a/1b38ac1a-71db-4ef7-b830-b2f3080e4569"
-					(reference "R74")
+					(reference "R73")
 					(unit 1)
 				)
@@
 		(on_board yes)
 		(dnp no)
-		(property "Reference" "#PWR086"
+		(property "Reference" "#PWR087"
 			(at 87.63 186.69 0)
 			(effects
@@
 			(project "CTS-SAT-2-OBC-PCB"
 				(path "/58243925-df8d-4fc1-899e-fce866d1d25a/1b38ac1a-71db-4ef7-b830-b2f3080e4569"
-					(reference "#PWR086")
+					(reference "#PWR087")
 					(unit 1)
 				)
@@
 		(dnp no)
 		(fields_autoplaced yes)
-		(property "Reference" "#PWR096"
+		(property "Reference" "#PWR097"
 			(at 160.02 185.42 0)
 			(effects
@@
 			(project "CTS-SAT-2-OBC-PCB"
 				(path "/58243925-df8d-4fc1-899e-fce866d1d25a/1b38ac1a-71db-4ef7-b830-b2f3080e4569"
-					(reference "#PWR096")
+					(reference "#PWR097")
 					(unit 1)
 				)
@@
 		(on_board yes)
 		(dnp no)
-		(property "Reference" "#PWR087"
+		(property "Reference" "#PWR088"
 			(at 87.63 226.06 0)
 			(effects
@@
 			(project "CTS-SAT-2-OBC-PCB"
 				(path "/58243925-df8d-4fc1-899e-fce866d1d25a/1b38ac1a-71db-4ef7-b830-b2f3080e4569"
-					(reference "#PWR087")
+					(reference "#PWR088")
 					(unit 1)
 				)
@@
 		(dnp no)
 		(fields_autoplaced yes)
-		(property "Reference" "#PWR097"
+		(property "Reference" "#PWR098"
 			(at 149.86 187.96 0)
 			(effects
@@
 			(project "CTS-SAT-2-OBC-PCB"
 				(path "/58243925-df8d-4fc1-899e-fce866d1d25a/1b38ac1a-71db-4ef7-b830-b2f3080e4569"
-					(reference "#PWR097")
+					(reference "#PWR098")
 					(unit 1)
 				)
@@
 		(dnp no)
 		(fields_autoplaced yes)
-		(property "Reference" "#PWR093"
+		(property "Reference" "#PWR094"
 			(at 149.86 109.22 0)
 			(effects
@@
 			(project "CTS-SAT-2-OBC-PCB"
 				(path "/58243925-df8d-4fc1-899e-fce866d1d25a/1b38ac1a-71db-4ef7-b830-b2f3080e4569"
-					(reference "#PWR093")
+					(reference "#PWR094")
 					(unit 1)
 				)
@@
 		(dnp no)
 		(fields_autoplaced yes)
-		(property "Reference" "#PWR091"
+		(property "Reference" "#PWR092"
 			(at 93.98 210.82 0)
 			(effects
@@
 			(project "CTS-SAT-2-OBC-PCB"
 				(path "/58243925-df8d-4fc1-899e-fce866d1d25a/1b38ac1a-71db-4ef7-b830-b2f3080e4569"
-					(reference "#PWR091")
+					(reference "#PWR092")
 					(unit 1)
 				)
@@
 		(on_board yes)
 		(dnp no)
-		(property "Reference" "R81"
+		(property "Reference" "R80"
 			(at 145.288 111.252 90)
 			(effects
@@
 			(project "CTS-SAT-2-OBC-PCB"
 				(path "/58243925-df8d-4fc1-899e-fce866d1d25a/1b38ac1a-71db-4ef7-b830-b2f3080e4569"
-					(reference "R81")
+					(reference "R80")
 					(unit 1)
 				)
@@
 		(dnp no)
 		(fields_autoplaced yes)
-		(property "Reference" "#PWR090"
+		(property "Reference" "#PWR091"
 			(at 93.98 171.45 0)
 			(effects
@@
 			(project "CTS-SAT-2-OBC-PCB"
 				(path "/58243925-df8d-4fc1-899e-fce866d1d25a/1b38ac1a-71db-4ef7-b830-b2f3080e4569"
-					(reference "#PWR090")
+					(reference "#PWR091")
 					(unit 1)
 				)
@@
 		(on_board yes)
 		(dnp no)
-		(property "Reference" "R77"
+		(property "Reference" "R76"
 			(at 97.282 111.252 90)
 			(effects
@@
 			(project "CTS-SAT-2-OBC-PCB"
 				(path "/58243925-df8d-4fc1-899e-fce866d1d25a/1b38ac1a-71db-4ef7-b830-b2f3080e4569"
-					(reference "R77")
+					(reference "R76")
 					(unit 1)
 				)
@@
 		(on_board yes)
 		(dnp no)
-		(property "Reference" "R78"
+		(property "Reference" "R77"
 			(at 97.282 149.352 90)
 			(effects
@@
 			(project "CTS-SAT-2-OBC-PCB"
 				(path "/58243925-df8d-4fc1-899e-fce866d1d25a/1b38ac1a-71db-4ef7-b830-b2f3080e4569"
-					(reference "R78")
-					(unit 1)
-				)
+					(reference "R77")
+					(unit 1)
+				)

Commit message: Assign footprints
Parts:
- C39, C40, C41, C42: footprint (none) -> Capacitor_SMD:C_0603_1608Metric
- IC2, IC3, IC4, IC5: footprint SOIC127P1030X265-16N -> Package_SO:SOIC-16W_7.5x10.3mm_P1.27mm
- R72, R73, R74, R75, R76, R77, R78, R79, R80, R81, R82, R83: footprint (none) -> Resistor_SMD:R_0603_1608Metric
Changed lines of the file:
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@@
 			)
 		)
-		(property "Footprint" "SOIC127P1030X265-16N"
+		(property "Footprint" "Package_SO:SOIC-16W_7.5x10.3mm_P1.27mm"
 			(at 142.24 265.1 0)
 			(effects
@@
 			)
 		)
-		(property "Footprint" ""
+		(property "Footprint" "Capacitor_SMD:C_0603_1608Metric"
 			(at 86.6648 93.98 0)
 			(effects
@@
 			)
 		)
-		(property "Footprint" ""
+		(property "Footprint" "Capacitor_SMD:C_0603_1608Metric"
 			(at 86.6648 132.08 0)
 			(effects
@@
 			)
 		)
-		(property "Footprint" ""
+		(property "Footprint" "Resistor_SMD:R_0603_1608Metric"
 			(at 101.346 186.944 90)
 			(effects
@@
 			)
 		)
-		(property "Footprint" "SOIC127P1030X265-16N"
+		(property "Footprint" "Package_SO:SOIC-16W_7.5x10.3mm_P1.27mm"
 			(at 142.24 304.47 0)
 			(effects
@@
 			)
 		)
-		(property "Footprint" ""
+		(property "Footprint" "Resistor_SMD:R_0603_1608Metric"
 			(at 100.076 178.054 90)
 			(effects
@@
 			)
 		)
-		(property "Footprint" ""
+		(property "Footprint" "Resistor_SMD:R_0603_1608Metric"
 			(at 100.076 217.424 90)
 			(effects
@@
 			)
 		)
-		(property "Footprint" ""
+		(property "Footprint" "Resistor_SMD:R_0603_1608Metric"
 			(at 101.346 226.314 90)
 			(effects
@@
 			)
 		)
-		(property "Footprint" ""
+		(property "Footprint" "Resistor_SMD:R_0603_1608Metric"
 			(at 100.076 99.314 90)
 			(effects
@@
 			)
 		)
-		(property "Footprint" ""
+		(property "Footprint" "Resistor_SMD:R_0603_1608Metric"
 			(at 150.114 148.336 90)
 			(effects
@@
 			)
 		)
-		(property "Footprint" ""
+		(property "Footprint" "Resistor_SMD:R_0603_1608Metric"
 			(at 150.114 228.346 90)
 			(effects
@@
 			)
 		)
-		(property "Footprint" ""
+		(property "Footprint" "Resistor_SMD:R_0603_1608Metric"
 			(at 150.114 188.976 90)
 			(effects
@@
 			)
 		)
-		(property "Footprint" "SOIC127P1030X265-16N"
+		(property "Footprint" "Package_SO:SOIC-16W_7.5x10.3mm_P1.27mm"
 			(at 142.24 186.36 0)
 			(effects
@@
 			)
 		)
-		(property "Footprint" ""
+		(property "Footprint" "Capacitor_SMD:C_0603_1608Metric"
 			(at 86.6648 172.72 0)
 			(effects
@@
 			)
 		)
-		(property "Footprint" ""
+		(property "Footprint" "Resistor_SMD:R_0603_1608Metric"
 			(at 100.076 137.414 90)
 			(effects
@@
 			)
 		)
-		(property "Footprint" ""
+		(property "Footprint" "Capacitor_SMD:C_0603_1608Metric"
 			(at 86.6648 212.09 0)
 			(effects
@@
 			)
 		)
-		(property "Footprint" ""
+		(property "Footprint" "Resistor_SMD:R_0603_1608Metric"
 			(at 150.114 110.236 90)
 			(effects
@@
 			)
 		)
-		(property "Footprint" ""
+		(property "Footprint" "Resistor_SMD:R_0603_1608Metric"
 			(at 101.346 108.204 90)
 			(effects
@@
 			)
 		)
-		(property "Footprint" "SOIC127P1030X265-16N"
+		(property "Footprint" "Package_SO:SOIC-16W_7.5x10.3mm_P1.27mm"
 			(at 142.24 224.46 0)
 			(effects
@@
 			)
 		)
-		(property "Footprint" ""
+		(property "Footprint" "Resistor_SMD:R_0603_1608Metric"
 			(at 101.346 146.304 90)
 			(effects
