File: Hardware/CTS-SAT-2-OBC-PCB.kicad_pcb (KiCad board)
At the start: 6 copper layers, 95.9 x 90.2 mm, 213 parts, among them IC1 STTS22HTR, IC2 MT29F1G01ABAFDSF-AAT_F_TR, IC3 MT29F1G01ABAFDSF-AAT_F_TR, IC4 MT29F1G01ABAFDSF-AAT_F_TR, IC5 MT29F1G01ABAFDSF-AAT_F_TR, J10 J-0532610871, J11 J-TSW-106-05-T-S, J12 J-0532610671, J13 J-0532610471, J14 J-0532610471, J15 J-TSW-106-05-T-S, J16 J-0532610671, J17 J-0532610471, J18 252105, J19 252105, J2 2-Pin Header, J20 252105, J21 J-0530471010, J22 J-0530471010, J23 J-0532610471, J24 USB_C_Receptacle_USB2.0_14P, J25 J-0532610471, J3 ESQ-126-14-G-D, J4 ESQ-126-14-G-D, J5 2-Pin Header, J6 2-Pin Header, J7 J-0532610671, J8 J-0532610471, J9 J-0532610871, SW1 SW_Push_Dual, SW2 SW_Push_Dual, U1 W25Q128JVS, U2 RP2040, U3 STM32L4R5ZITx, U4 SN74LVC1G14DCKR, U5 HMC544AE, U6 U-MAX3378EEUD+T, U7 MAX3086EESD+T, Y1 ABM8-272-T3, Y2 TG-3541CE_32.7680KXB3, Y3 ECS-TXO-2520-33-250-AN-TR

Commit message: Refill zones
Parts:
- moved R24 1.82 mm to (119.2, 91.4)
- moved R28 1.33 mm to (118.1, 99.8)
- moved R30 1.33 mm to (118.1, 101.2)
- moved R25 1.08 mm to (117.9, 95.2)
- moved R26 1.08 mm to (117.9, 96.8)
- moved R27 1.08 mm to (117.9, 98.2)
Routing:
- net Net-(U3-PD6): track 5.06 -> 3.73 mm
- net Net-(U3-PD3): track 4.75 -> 3.68 mm
- net Net-(U3-PD2): track 4.34 -> 3.26 mm
- net Net-(U3-PD1): track 4.75 -> 3.68 mm
- net Net-(U3-PD4): track 5.27 -> 4.32 mm
- net Net-(U3-PA15): track 5.81 -> 5.00 mm

Commit message: Begin routing
Parts:
- moved J15 18.2 mm to (182.5, 96.4)
- moved J16 17.5 mm to (192.3, 89.9)
- moved R69 17.5 mm to (187.3, 91.7)
- moved R70 17.5 mm to (187.2, 89.7)
- moved R71 17.5 mm to (187.1, 87.9)
- moved J11 14.1 mm to (182.4, 112.3)
- moved J12 14.1 mm to (192.2, 106.0)
- moved R65 14.1 mm to (187.2, 107.8)
- moved R66 14.1 mm to (187.1, 106.0)
- moved R67 14.1 mm to (187.1, 104.3)
- moved R68 14.1 mm to (187.2, 102.5)
Connections:
- J11 pad 01: 3V3 -> +3V3
- J12 pad 1: 3V3 -> +3V3
- J15 pad 01: 3V3 -> +3V3
- J16 pad 1: 3V3 -> +3V3
- R58 pad 2: 3V3 -> +3V3
- R60 pad 2: 3V3 -> +3V3
- U4 pad 1: Net-(U4-NC) -> unconnected-(U4-NC-Pad1)
Routing:
- net 12V_MPI: track 0.00 -> 78.3 mm, vias 0 -> 1
- net /Connectors/STM32_SWCLK: track 4.75 -> 82.6 mm, vias 0 -> 1
- net /Connectors/STM32_SWDIO: track 4.41 -> 74.6 mm, vias 0 -> 1
- net /Connectors/RP2040_NRST: track 4.15 -> 72.9 mm, vias 0 -> 2
- net /Connectors/RP2040_SWCLK: track 5.15 -> 73.0 mm, vias 0 -> 2
- net /Connectors/RP2040_SWDIO: track 3.87 -> 67.9 mm, vias 0 -> 1
- net /Connectors/STM32_SWO: track 5.19 -> 67.9 mm, vias 0 -> 1
- net +3V3: track 79.2 -> 133.6 mm, vias 2 -> 35
- net /Connectors/STM32_NRST: track 10.5 -> 62.2 mm, vias 0 -> 1
- net GND: track 241.0 -> 262.1 mm, vias 45 -> 62
- net 3V3: track 23.9 -> 6.10 mm
- net /Antenna/3V3_ANT_DEPLOY: track 7.00 -> 13.9 mm
- net Net-(U3-PA5): track 0.00 -> 4.54 mm, vias 0 -> 2
- net Net-(U3-PA7): track 0.00 -> 3.68 mm, vias 0 -> 2
- net Net-(U3-PC5): track 0.00 -> 3.59 mm
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- added copper zone on In3.Cu, net +3V3

Commit message: Continue routing
Parts:
- removed the R26 at (111.2, 132.0)
- removed the R30 at (179.8, 58.5)
Connections:
- R55 pad 1: V_BAT -> +BATT
Routing:
- net /Memory/SPI_FLASH_MOSI: track 0.00 -> 117.5 mm, vias 0 -> 5
- net /Memory/SPI_FLASH_SCLK: track 0.00 -> 114.6 mm, vias 0 -> 5
- net /Connectors/MISO_USART2_RX: track 2.69 -> 99.8 mm, vias 0 -> 2
- net /Memory/SPI_FLASH_MISO: track 0.00 -> 56.9 mm, vias 0 -> 2
- net Net-(U3-PC12): track 0.00 -> 40.4 mm, vias 0 -> 2
- net /Connectors/MISO_UART5_RX: track 2.42 -> 40.6 mm, vias 0 -> 2
- net Net-(U2-USB_DM): track 2.01 -> 36.5 mm, vias 1 -> 2
- net Net-(U2-USB_DP): track 1.27 -> 34.2 mm, vias 1 -> 2
- net /Connectors/RP2040_NRST: track 72.9 -> 91.5 mm
- net GND: track 262.1 -> 275.1 mm, vias 62 -> 65
- net +3V3: track 133.6 -> 138.3 mm, vias 35 -> 39
- net /Connectors/RP2040_SWDIO: track 67.9 -> 72.6 mm
- net /Memory/SPI_NCS_FLASH_2: track 4.34 -> 8.43 mm, vias 0 -> 1
- net /RP2040/SPI1_RX: track 1.67 -> 5.28 mm, vias 1 -> 2
- net Net-(U3-PD5): track 0.00 -> 3.53 mm, vias 0 -> 2
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
Commit message: Replace Optical Downlink with ADCS Sensors connector
Parts:
- removed J17: J-0532610471, CTS-SAT-1:J-53261-0471
- removed R29: 22R, Resistor_SMD:R_0603_1608Metric
- removed R30: 0R, Resistor_SMD:R_0603_1608Metric
- added J1: J-0530471010, CTS-SAT-1:J-0530471010, F.Cu at (177.0, 52.8)
Routing:
- net /Connectors/MISO_USART2_RX: track 99.8 -> 6.54 mm, vias 2 -> 1
- net GND: track 275.1 -> 264.5 mm, vias 65 -> 63
- net +3V3: track 138.3 -> 134.0 mm
- net /Connectors/MOSI_USART2_TX: track 2.45 -> 0.00 mm
- net Net-(U3-PD5): track 3.53 -> 1.99 mm, vias 2 -> 1
Other:
- board text added: "ADCS Sensors"
- board text removed: "Optical Downlink"
