File: Hardware/STM32.kicad_sch (KiCad schematic)
At the start: 74 parts, among them IC1 STTS22HTR, SW1 SW_Push_Dual, U3 STM32L4R5ZITx, Y2 TG-3541CE_32.7680KXB3, Y3 ECS-TXO-2520-33-250-AN-TR

Commit message: Adjust schematic for new ADC pins
Connections:
- net ADCS_CSS_1: now also U3.40 (PA4)
- net ADCS_CSS_2: now also U3.41 (PA5)
- net ADCS_CSS_3: now also U3.42 (PA6)
- net ADCS_CSS_4: now also U3.43 (PA7)
- net ADCS_CSS_5: now also U3.46 (PB0)
- net ADCS_CSS_6: now also U3.47 (PB1)
- net ADCS_FSS_1: now also U3.36 (PA2)
- net ADCS_FSS_2: now also U3.37 (PA3)
- net ADCS_MTM_IN: now also U3.29 (PC3)
- net at R16.1: now also U3.48 (PB2); no longer U3.37 (PA3)
- net at R18.2: now also U3.53 (PF13); no longer U3.42 (PA6)
- net at R17.1: now also U3.49 (PF11); no longer U3.40 (PA4)
- net at R100.1: now also U3.50 (PF12); no longer U3.41 (PA5)
- net at U3.22 (PF10): now also R15.1
- net at R101.1: now also U3.54 (PF14); no longer U3.43 (PA7)
- no-connect marks 70 -> 61
Other:
- moved on the sheet: R100, R101, R15, R16, R17, R18

Commit message: finish routing!
Connections:
- net STM_UHF_CTL: now also U3.63 (PE10)
- no-connect marks 61 -> 60
Changed lines of the file:
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@@
 	)
 	(no_connect
-		(at 247.65 208.28)
-	)
-	(no_connect
 		(at 107.95 180.34)
 	)
@@
 	(wire
 		(pts
-			(xy 173.99 54.61) (xy 181.61 54.61)
+			(xy 255.27 208.28) (xy 247.65 208.28)
 		)
 		(stroke
@@
 	(hierarchical_label "STM_UHF_CTL"
 		(shape output)
-		(at 173.99 54.61 180)
+		(at 255.27 208.28 0)
 		(effects
 			(font
 				(size 1.27 1.27)
 			)
-			(justify right)
+			(justify left)
 		)
 	)

Commit message: Fix the switches
Connections:
- net GND: now also SW1.3, SW1.4; no longer SW1.2
- net at R48.2, SW1.1: now also SW1.2
Changed lines of the file:
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@@
 		(on_board yes)
 		(dnp no)
-		(fields_autoplaced yes)
 		(property "Reference" "SW1"
-			(at 307.34 63.5 0)
+			(at 307.594 66.294 0)
 			(effects
 				(font
@@
 					(size 1.27 1.27)
 				)
+				(hide yes)
 			)
 		)
@@
 		(pin "1"
 		)
+		(pin "3"
+		)
+		(pin "4"
+		)
 		(pin "2"
